Commit message: added dummy inertia to hexapod joint entries

File: robot-graphics/robot-graphics/URDF/hexapod.urdf (robot description, URDF)
Before this commit: robot ability_hand, 19 links, 18 joints
Links:
- link leg1_link1: mass None -> 0.1
- link leg1_link2: mass None -> 0.1
- link leg1_link3: mass None -> 0.1
- link leg2_link1: mass None -> 0.1
- link leg2_link2: mass None -> 0.1
- link leg2_link3: mass None -> 0.1
- link leg3_link1: mass None -> 0.1
- link leg3_link2: mass None -> 0.1
- link leg3_link3: mass None -> 0.1
- link leg4_link1: mass None -> 0.1
- link leg4_link2: mass None -> 0.1
- link leg4_link3: mass None -> 0.1
- link leg5_link1: mass None -> 0.1
- link leg5_link2: mass None -> 0.1
- link leg5_link3: mass None -> 0.1
- link leg6_link1: mass None -> 0.1
- link leg6_link2: mass None -> 0.1
- link leg6_link3: mass None -> 0.1
